Commit message: Añadido jaguar cpp, arreglados errores en teleop_jaguar.cpp y añadidos dos mundos

File: ROS/jaguar_ros/urdf/model.urdf (robot description, URDF)
Before this commit: robot jaguar, 10 links, 9 joints
Links:
- added link ir_base, mass 0.001; visual box size=0.001 0.001 0.001
Joints:
- added joint ir_joint: type fixed, parent base_link, child ir_base, origin xyz=0.3 0 0.03 rpy=0 1.57 0, axis 1 0 0
- joint velodyne_base_j: origin xyz=0  0  0.5 rpy=0      0     0 -> xyz=0  0  0.2 rpy=0      0     0

Commit message: Añadido repo Karim y modificados pcl_staris y teleop_jaguar y teleop_jaguar.launch

File: ROS/jaguar_ros/urdf/model.urdf (robot description, URDF)
Before this commit: robot jaguar, 11 links, 10 joints
Links:
- added link ir_front, mass 0.001; visual box size=0.001 0.001 0.001
Joints:
- added joint ir_front_joint: type fixed, parent base_link, child ir_front, origin xyz=0.3 0 0.04 rpy=0 0 0, axis 1 0 0
